Commit message: Add shopping cart to SARA's URDF and fix Gazebo spawn/TF issues

File: sara_description/models/sara.gazebo.xacro (robot description, xacro)
@@ -1,8 +1,37 @@
 <?xml version="1.0"?>
-<robot name="turtlebot3_burger_sim" xmlns:xacro="http://ros.org/wiki/xacro">
+<robot name="sara_sim" xmlns:xacro="http://ros.org/wiki/xacro">
   <xacro:arg name="laser_visual" default="false"/>
   <xacro:arg name="imu_visual"   default="false"/>
   <gazebo reference="base_link">
     <material>Gazebo/DarkGrey</material>
+  </gazebo>
+  <!-- sdformat's urdf2sdf multiplies each URDF <material><color> by 1.25 when
+       converting to SDF, which clips/shifts colors (e.g. 0.894 grey -> 1.0
+       white). These overrides set gz-sim's ambient/diffuse directly, bypassing
+       that conversion, so Gazebo matches the true SolidWorks colors used in
+       sara.urdf.xacro/RViz instead of the shifted ones. -->
+  <gazebo reference="base_cart">
+    <visual>
+      <material>
+        <ambient>0.86667 0.32157 0.15686 1</ambient>
+        <diffuse>0.86667 0.32157 0.15686 1</diffuse>
+      </material>
+    </visual>
+  </gazebo>
+  <gazebo reference="base_platform">
+    <visual>
+      <material>
+        <ambient>0.55 0.55 0.55 1</ambient>
+        <diffuse>0.55 0.55 0.55 1</diffuse>
+      </material>
+    </visual>
+  </gazebo>
+  <gazebo reference="base_weight">
+    <visual>
+      <material>
+        <ambient>1 1 1 1</ambient>
+        <diffuse>1 1 1 1</diffuse>
+      </material>
+    </visual>
   </gazebo>
   <gazebo reference="wheel_left_link">

File: sara_description/models/sara.urdf.xacro (robot description, xacro)
@@ -1,4 +1,4 @@
 <?xml version="1.0" ?>
-<robot name="turtlebot3_burger" xmlns:xacro="http://ros.org/wiki/xacro">
+<robot name="sara" xmlns:xacro="http://ros.org/wiki/xacro">
   <xacro:include filename="$(find sara_description)/models/common_properties.xacro"/>
   <xacro:include filename="$(find sara_description)/models/sara.gazebo.xacro"/>
@@ -185,3 +185,102 @@
   </joint>
   <link name="camera_rgb_optical_frame"/>
+  <!-- Shopping cart superstructure, mounted flush with the top of the chassis deck.
+       x=-0.064 matches the chassis mesh/scan_joint offset: base_link's origin is the wheel
+       axle, not the visual center of the round plate, which sits 0.064m behind it.
+       z=0.0915 is the top of waffle_pi_base.stl itself (91.5mm tall, scale 0.001), i.e. the
+       standoffs (base_cart) start right at the deck surface, not artificially raised to
+       clear the LIDAR (which sits off-center at x=-0.064 too, so it doesn't collide with
+       the corner-mounted standoffs anyway). -->
+  <joint name="cart_mount_joint" type="fixed">
+    <parent link="base_link"/>
+    <child link="base_cart"/>
+    <origin xyz="-0.064 0.0 0.0915" rpy="0 0 0"/>
+  </joint>
+  <link name="base_cart">
+    <inertial>
+      <origin xyz="0.00029076 0.0018904 0.0225" rpy="0 0 0"/>
+      <mass value="0.0034946"/>
+      <inertia ixx="5.3922E-07" ixy="6.2156E-23" ixz="1.2408E-23"
+               iyy="5.3922E-07" iyz="1.8924E-21"
+               izz="1.322E-08"/>
+    </inertial>
+    <visual>
+      <origin xyz="0 0 0" rpy="0 0 0"/>
+      <geometry>
+        <mesh filename="package://sara_description/meshes/cart/base_cart.STL"/>
+      </geometry>
+      <material name="cart_orange">
+        <color rgba="0.86667 0.32157 0.15686 1"/>
+      </material>
+    </visual>
+    <collision>
+      <origin xyz="0 0 0" rpy="0 0 0"/>
+      <geometry>
+        <mesh filename="package://sara_description/meshes/cart/base_cart.STL"/>
+      </geometry>
+    </collision>
+  </link>
+  <joint name="cart_platform_joint" type="fixed">
+    <parent link="base_cart"/>
+    <child link="base_platform"/>
+    <origin xyz="0 0 0.041" rpy="0 0 0"/>
+  </joint>
+  <link name="base_platform">
+    <inertial>
+      <origin xyz="0.0037131 0.00016219 0.044512" rpy="0 0 0"/>
+      <mass value="1.4652"/>
+      <inertia ixx="0.0032997" ixy="8.2131E-06" ixz="-5.2149E-06"
+               iyy="0.0030443" iyz="-1.1568E-06"
+               izz="0.0037989"/>
+    </inertial>
+    <visual>
+      <origin xyz="0 0 0" rpy="0 0 0"/>
+      <geometry>
+        <mesh filename="package://sara_description/meshes/cart/Base_platform.STL"/>
+      </geometry>
+      <!-- Base_platform is a merged multi-part assembly (scale/load-cell base,
+           the basket, the display case, and a mounting plate) collapsed into
+           one mesh by the SW export, with no per-part color data preserved.
+           Using the original exported appearance (grey) instead of guessing
+           a single color for the whole assembly. -->
+      <material name="cart_grey">
+        <color rgba="0.55 0.55 0.55 1"/>
+      </material>
+    </visual>
+    <collision>
+      <origin xyz="0 0 0" rpy="0 0 0"/>
+      <geometry>
+        <mesh filename="package://sara_description/meshes/cart/Base_platform.STL"/>
+      </geometry>
+    </collision>
+  </link>
+  <joint name="cart_weight_joint" type="fixed">
+    <parent link="base_platform"/>
+    <child link="base_weight"/>
+    <origin xyz="0.015647 0 0.0552" rpy="0 0 0"/>
+  </joint>
+  <link name="base_weight">
+    <inertial>
+      <origin xyz="0.00067058 -1.299E-14 -0.0051801" rpy="0 0 0"/>
+      <mass value="0.19409"/>
+      <inertia ixx="0.00032968" ixy="8.3723E-15" ixz="1.2781E-06"
+               iyy="0.0007598" iyz="-2.6448E-17"
+               izz="0.0010856"/>
+    </inertial>
+    <visual>
+      <origin xyz="0 0 0" rpy="0 0 0"/>
+      <geometry>
+        <mesh filename="package://sara_description/meshes/cart/Base_weight.STL"/>
+      </geometry>
+      <material name="cart_white">
+        <color rgba="1 1 1 1"/>
+      </material>
+    </visual>
+    <collision>
+      <origin xyz="0 0 0" rpy="0 0 0"/>
+      <geometry>
+        <mesh filename="package://sara_description/meshes/cart/Base_weight.STL"/>
+      </geometry>
+    </collision>
+  </link>
 </robot>

Commit message: Add simulated weight sensor and implement Payload Interaction mode
- Add a force_torque sensor at cart_weight_joint (base_platform ->
  base_weight, the real load cell's location per the SolidWorks assembly).
  Required converting that joint from fixed to prismatic (near-zero range,
  stiff spring): gz-sim's ForceTorque system only attaches to joints with
  an axis, and dartsim (the container's physics engine) can't build mesh
  collisions, so the cart links also get box collision primitives sized
  from their STL bounding boxes.
- Bridge cart_weight_wrench to ROS and add sara_safety/weight_monitor.py,
  implementing Payload Interaction (paper2_draft.md S3.3) as specified:
  a soft rate-of-change (dW/dt) trigger for temporary speed reduction plus
  a warning flag, and a hard absolute-weight trigger for an immediate stop
  via cmd_vel_block_all (twist_mux priority 255, same mechanism as the
  real robot's mux_locker.py). Wired into both sara.launch.py and
  sara_safety/mux.launch.py.
- Add effort/velocity limits to the wheel joints, sourced from the real
  TB3 Waffle Pi's DYNAMIXEL XM430-W210 datasheet (3.0 N.m stall, 8.06
  rad/s no-load). Without these, gz-sim's velocity controller could apply
  unlimited torque, so payload mass had no effect on acceleration/braking
  at all - verified empirically after the fix (max speed now correctly
  caps at the real Waffle's ~0.266 m/s; braking measurably slower loaded).
- speed_limit.py now scales its max linear/angular speed by
  cart_speed_scale instead of using fixed constants.

File: sara_description/models/sara.gazebo.xacro (robot description, xacro)
@@ -99,4 +99,25 @@
       <topic>joint_states</topic>
     </plugin>
+    <!-- Required for any <sensor type="force_torque"> to actually produce
+         output (cart_weight_joint below) - it's a separate system from
+         Physics/Sensors, must be loaded explicitly like DiffDrive/JSP above. -->
+    <plugin filename="gz-sim-forcetorque-system" name="gz::sim::systems::ForceTorque">
+    </plugin>
+  </gazebo>
+  <!-- Weight sensor: cart_weight_joint is where the physical design's load
+       cell actually sits (base_weight = "TopeBascula", the load cell's
+       contact plate; base_platform = the fixed side it presses against per
+       the SolidWorks assembly). Reports the support-reaction wrench, i.e.
+       the weight of everything resting on base_weight. -->
+  <gazebo reference="cart_weight_joint">
+    <sensor name="cargo_scale" type="force_torque">
+      <always_on>true</always_on>
+      <update_rate>20</update_rate>
+      <topic>cart_weight_wrench</topic>
+      <force_torque>
+        <frame>child</frame>
+        <measure_direction>child_to_parent</measure_direction>
+      </force_torque>
+    </sensor>
   </gazebo>
   <gazebo reference="base_scan">

File: sara_description/models/sara.urdf.xacro (robot description, xacro)
@@ -31,4 +31,10 @@
     </inertial>
   </link>
+  <!-- effort/velocity from the real TB3 Waffle Pi's DYNAMIXEL XM430-W210
+       datasheet (3.0 N.m stall torque at 12V, 77 RPM = 8.06 rad/s no-load).
+       Without an effort limit, gz-sim's DiffDrive velocity controller can
+       apply unlimited torque to hit the commanded wheel speed regardless of
+       load, which would make added cargo mass have no effect on the robot's
+       acceleration - the opposite of what Payload Interaction needs to show. -->
   <joint name="wheel_left_joint" type="continuous">
     <parent link="base_link"/>
@@ -36,4 +42,5 @@
     <origin xyz="0.0 0.144 0.023" rpy="-1.57 0 0"/>
     <axis xyz="0 0 1"/>
+    <limit effort="3.0" velocity="8.06"/>
   </joint>
   <link name="wheel_left_link">
@@ -64,4 +71,5 @@
     <origin xyz="0.0 -0.144 0.023" rpy="-1.57 0 0"/>
     <axis xyz="0 0 1"/>
+    <limit effort="3.0" velocity="8.06"/>
   </joint>
   <link name="wheel_right_link">
@@ -214,8 +222,14 @@
       </material>
     </visual>
-    <collision>
-      <origin xyz="0 0 0" rpy="0 0 0"/>
-      <geometry>
-        <mesh filename="package://sara_description/meshes/cart/base_cart.STL"/>
+    <!-- Box approximation of the mesh, not the mesh itself: dartsim (used by
+         the sara_jazzy container's default physics config) can't construct
+         collision geometry from a mesh yet ("Mesh construction from an SDF
+         has not been implemented yet for dartsim"), so a mesh collision here
+         silently disappears under it - dropped objects would fall straight
+         through. Sized/centered from the STL's own bounding box. -->
+    <collision>
+      <origin xyz="0.0013 0.0020 0.0225" rpy="0 0 0"/>
+      <geometry>
+        <box size="0.1635 0.2585 0.0450"/>
       </geometry>
     </collision>
@@ -248,15 +262,29 @@
       </material>
     </visual>
-    <collision>
-      <origin xyz="0 0 0" rpy="0 0 0"/>
-      <geometry>
-        <mesh filename="package://sara_description/meshes/cart/Base_platform.STL"/>
-      </geometry>
-    </collision>
-  </link>
-  <joint name="cart_weight_joint" type="fixed">
+    <!-- Box approximation, see base_cart's collision comment above. Only the
+         bottom ~3cm (the structural floor), not the mesh's full 0.146m
+         height: that height is mostly hollow basket wall, and a full-height
+         solid box would fill the whole cavity, blocking anything from ever
+         reaching base_weight's pad inside it. -->
+    <collision>
+      <origin xyz="-0.0173 0.0000 0.015" rpy="0 0 0"/>
+      <geometry>
+        <box size="0.3150 0.2655 0.03"/>
+      </geometry>
+    </collision>
+  </link>
+  <!-- Modeled as prismatic (not fixed) with a near-zero range and a stiff
+       spring: this is how the real load cell actually works (the contact
+       plate deflects a tiny amount under load, which is what the strain
+       gauge measures), and gz-sim's ForceTorque sensor system only attaches
+       to joints with an axis/DOF - a fixed joint has none, so the sensor
+       would silently produce no output. -->
+  <joint name="cart_weight_joint" type="prismatic">
     <parent link="base_platform"/>
     <child link="base_weight"/>
     <origin xyz="0.015647 0 0.0552" rpy="0 0 0"/>
+    <axis xyz="0 0 1"/>
+    <limit lower="-0.0005" upper="0.0005" effort="100" velocity="0.01"/>
+    <dynamics damping="50.0" friction="0.0"/>
   </joint>
   <link name="base_weight">
@@ -277,8 +305,9 @@
       </material>
     </visual>
-    <collision>
-      <origin xyz="0 0 0" rpy="0 0 0"/>
-      <geometry>
-        <mesh filename="package://sara_description/meshes/cart/Base_weight.STL"/>
+    <!-- Box approximation, see base_cart's collision comment above -->
+    <collision>
+      <origin xyz="-0.0017 0.0000 -0.0100" rpy="0 0 0"/>
+      <geometry>
+        <box size="0.2280 0.1480 0.0200"/>
       </geometry>
     </collision>

Commit message: add collaborative operating modes

File: sara_description/models/sara.gazebo.xacro (robot description, xacro)
@@ -60,7 +60,16 @@
     <material>Gazebo/FlatBlack</material>
   </gazebo>
-  <gazebo reference="caster_back_link">
-    <mu1>0.1</mu1>
-    <mu2>0.1</mu2>
+  <gazebo reference="caster_back_right_link">
+    <mu1>0.4</mu1>
+    <mu2>0.4</mu2>
+    <kp>1000000.0</kp>
+    <kd>100.0</kd>
+    <minDepth>0.001</minDepth>
+    <maxVel>1.0</maxVel>
+    <material>Gazebo/FlatBlack</material>
+  </gazebo>
+  <gazebo reference="caster_back_left_link">
+    <mu1>0.4</mu1>
+    <mu2>0.4</mu2>
     <kp>1000000.0</kp>
     <kd>100.0</kd>
